Commit message: full simulation version of rosbot

File: description/body.urdf.xacro (robot description, xacro)
@@ -31,5 +31,9 @@
     </link>
     <gazebo reference="body_link">
-      <material>Gazebo/White</material>
+      <visual>
+          <material>
+              <script>Gazebo/White</script>
+          </material>
+      </visual>
     </gazebo>
     <joint name="body_to_cover_joint" type="fixed">
@@ -49,5 +53,9 @@
       </visual>
       <gazebo reference="cover_link">
-        <material>Gazebo/Red</material>
+          <visual>
+              <material>
+                  <script>Gazebo/Red</script>
+              </material>
+          </visual>
       </gazebo>
       <inertial>

File: description/rosbot.urdf.xacro (robot description, xacro)
@@ -2,19 +2,16 @@
 <robot name="rosbot" xmlns:xacro="http://www.ros.org/wiki/xacro">
   <xacro:arg name="use_sim" default="true" />
-  <xacro:arg name="use_gpu" default="true" />
-  <xacro:arg name="simulation_engine" default="gazebo" />
-   <!-- <xacro:include filename="$(find rosbot_description)/urdf/rosbot_macro.urdf.xacro" ns="husarion" /> -->
-  <xacro:include filename="$(find rosbot)/description/rosbot_macro.urdf.xacro" ns="rosbot" />
+  <xacro:arg name="simulation_engine" default="gazebo-classic" />
+  <xacro:arg name="husarion_ros_build_type" default="simulation" />
+   <xacro:include filename="$(find rosbot)/description/rosbot_macro.urdf.xacro" ns="rosbot" />
   <xacro:rosbot.rosbot_robot use_sim="$(arg use_sim)" simulation_engine="$(arg simulation_engine)"/>
-   <!-- <xacro:include filename="$(find rosbot_description)/urdf/ros2_control.xacro"/> -->
   <xacro:include filename="$(find rosbot)/description/ros2_control.xacro"/>
-  <xacro:include filename="$(find ros_components_description)/urdf/slamtec_rplidar_a2.urdf.xacro" ns="lidar" />
+   <xacro:include filename="$(find rosbot)/description/slamtec_rplidar_a2.urdf.xacro" ns="lidar" />
   <xacro:lidar.slamtec_rplidar_a2
     parent_link="cover_link"
     xyz="0.02 0.0 0.0"
     rpy="0.0 0.0 0.0"
-    use_gpu="$(arg use_gpu)"
     simulation_engine="$(arg simulation_engine)" />
-  <xacro:include filename="$(find ros_components_description)/urdf/orbbec_astra.urdf.xacro" ns="camera" />
+  <xacro:include filename="$(find rosbot)/description/orbbec_astra.urdf.xacro" ns="camera" />
   <xacro:camera.orbbec_astra
     parent_link="camera_link"

Commit message: base_footprint now set up

File: description/body.urdf.xacro (robot description, xacro)
@@ -3,4 +3,10 @@
   <!-- body defining macro -->
   <xacro:macro name="body" params="wheel_radius">
+    <link name="base_footprint" />
+    <joint name="base_footprint_joint" type="fixed">
+          <origin xyz="0.0 0.0 0.0" rpy="0.0 0.0 0.0" />
+          <parent link="base_footprint" />
+          <child link="base_link" />
+    </joint>
     <link name="base_link" />
     <joint name="base_to_body_joint" type="fixed">

File: description/rosbot_macro.urdf.xacro (robot description, xacro)
@@ -78,5 +78,14 @@
             <publish_wheel_tf>true</publish_wheel_tf>
             <odometry_frame>odom</odometry_frame>
-            <robot_base_frame>base_link</robot_base_frame>
+            <!-- <robot_base_frame>base_link</robot_base_frame> -->
+            <robot_base_frame>base_footprint</robot_base_frame>
+          </plugin>
+          <plugin filename="libgazebo_ros_p3d.so" name="gazebo_ros_p3d">
+              <body_name>base_footprint</body_name>
+              <always_on>true</always_on>
+              <update_rate>100.0</update_rate>
+              <ros>
+                <remapping>odom:=ground_truth_odom</remapping>
+              </ros>
           </plugin>
         </gazebo>
